Commit message: eclass files
camera and myarm files

File: project_3/myarm/urdf/myarm_300_pi.urdf (robot description, URDF)
Before this commit: robot myarm_300_pi, 9 links, 8 joints
Links:
- link base: geometry collision mesh filename=../meshes/base.dae; visual mesh filename=../meshes/base.dae
- link link1: geometry collision mesh filename=../meshes/j1.dae; visual mesh filename=../meshes/j1.dae
- link link2: geometry collision mesh filename=../meshes/j2.dae; visual mesh filename=../meshes/j2.dae
- link link3: geometry collision mesh filename=../meshes/j3.dae; visual mesh filename=../meshes/j3.dae
- link link4: geometry collision mesh filename=../meshes/j4.dae; visual mesh filename=../meshes/j4.dae
- link link5: geometry collision mesh filename=../meshes/j5.dae; visual mesh filename=../meshes/j5.dae
- link link6: geometry collision mesh filename=../meshes/j6.dae; visual mesh filename=../meshes/j6.dae
- link link7: geometry collision mesh filename=../meshes/j7.dae; visual mesh filename=../meshes/j7.dae
Joints:
- joint link7_to_endeffector: origin xyz=0 0.0 0 rpy=0 0 0 -> xyz=0 0 0 rpy=0 0 0
